File: template/stencil/stencil.kicad_pcb (KiCad board)
At the start: 4 copper layers, 225 x 315 mm, 0 parts

Commit message: Update to KiCad 7.0
Other:
- outline, holes or cut-outs redrawn
- board text added: "locked"
Changed lines of the file:
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@@
-(kicad_pcb (version 20211014) (generator pcbnew)
+(kicad_pcb (version 20221018) (generator pcbnew)
   (general
     (thickness 1.6062)
   )
-  (paper "A4" portrait)
+  (paper "User" 224.993 315.011)
   (title_block
-    (date "2023-01-03")
+    (date "2023-01-11")
   )
   (layers
@@
   (setup
     (stackup
-      (layer "F.SilkS" (type "Top Silk Screen") (color "White"))
+      (layer "F.SilkS" (type "Top Silk Screen") (color "White") (color "White"))
       (layer "F.Paste" (type "Top Solder Paste"))
-      (layer "F.Mask" (type "Top Solder Mask") (color "Black") (thickness 0.01))
+      (layer "F.Mask" (type "Top Solder Mask") (color "Black") (color "Black") (thickness 0.01))
       (layer "F.Cu" (type "copper") (thickness 0.035))
       (layer "dielectric 1" (type "core") (thickness 0.2104) (material "FR4") (epsilon_r 4.5) (loss_tangent 0.02))
@@
       (layer "dielectric 3" (type "core") (thickness 0.2104) (material "FR4") (epsilon_r 4.5) (loss_tangent 0.02))
       (layer "B.Cu" (type "copper") (thickness 0.035))
-      (layer "B.Mask" (type "Bottom Solder Mask") (color "Black") (thickness 0.01))
+      (layer "B.Mask" (type "Bottom Solder Mask") (color "Black") (color "Black") (thickness 0.01))
       (copper_finish "HAL lead-free")
       (dielectric_constraints no)
     )
     (pad_to_mask_clearance 0)
-    (grid_origin 0 297)
+    (grid_origin 0 315)
     (pcbplotparams
       (layerselection 0x00010e8_ffffffff)
+      (plot_on_all_layers_selection 0x0000000_00000000)
       (disableapertmacros false)
       (usegerberextensions true)
@@
       (usegerberadvancedattributes false)
       (creategerberjobfile false)
-      (svguseinch false)
+      (dashed_line_dash_ratio 12.000000)
+      (dashed_line_gap_ratio 3.000000)
       (svgprecision 6)
-      (excludeedgelayer true)
       (plotframeref false)
       (viasonmask false)
@@
   )
   (net 0 "")
-  (gr_line (start 0 -17) (end 0 296) (layer "Edge.Cuts") (width 0.05))
-  (gr_line (start 1 -18) (end 224 -18) (layer "Edge.Cuts") (width 0.05))
-  (gr_line (start 225 -17) (end 225 296) (layer "Edge.Cuts") (width 0.05))
-  (gr_arc (start 1 297) (mid 0.292893 296.707107) (end 0 296) (layer "Edge.Cuts") (width 0.05))
-  (gr_arc (start 225 296) (mid 224.707107 296.707107) (end 224 297) (layer "Edge.Cuts") (width 0.05))
-  (gr_arc (start 0 -17) (mid 0.292893 -17.707107) (end 1 -18) (layer "Edge.Cuts") (width 0.05))
-  (gr_arc (start 224 -18) (mid 224.707107 -17.707107) (end 225 -17) (layer "Edge.Cuts") (width 0.05))
-  (gr_line (start 1 297) (end 224 297) (layer "Edge.Cuts") (width 0.05))
+  (gr_rect locked (start 0 0) (end 225 315)
+    (stroke (width 0.2) (type default)) (fill none) (layer "Edge.Cuts"))
+  (gr_line locked (start 112.5 302.5) (end 112.5 12.5)
+    (stroke (width 0.2) (type dash)) (layer "F.Fab"))
+  (gr_rect locked (start 17.5 12.5) (end 207.5 302.5)
+    (stroke (width 0.2) (type solid)) (fill none) (layer "F.Fab"))
+  (gr_line locked (start 207.5 157.5) (end 17.5 157.5)
+    (stroke (width 0.2) (type dash)) (layer "F.Fab"))
+  (gr_text locked "190 x 290" (at 184.5 308) (layer "F.Fab")
+    (effects (font (size 3 3) (thickness 0.15)) (justify left bottom))
+  )
+  (gr_text locked "225 x 315" (at 202 320.75) (layer "F.Fab")
+    (effects (font (size 3 3) (thickness 0.15)) (justify left bottom))
+  )
 )
